File: KiCad/AT386SX.kicad_pcb (KiCad board)
At the start: 2 copper layers, 218.4 x 167.6 mm, 130 parts, among them J1 KEYBOARD, J10 OSC_PIN1, J11 OSC_PIN8, J2 BUSAT_HOST, J3 BUSAT_HOST, J4 BUSAT_HOST, J5 BUSAT_HOST, J6 BUSAT_HOST, J7 BUSAT_HOST, J8 AT_POWER1, J9 AT_POWER2, Q3 2N3904, U1 8242KBD, U10 BANK0, U11 BANK0, U12 BANK1, U13 BANK1, U2 74HC05, U3 SST39SF010A, U4 DS12885, U6 ICW42C07, U7 Cx486SLC, U8 80387SX, U9 RC2016A5, X1 32768Hz, X2 14.31818MHz

Commit message: Version 1.3: Implement PS/2 mouse. Use PS/2 dualport pinout for the keyboard/mouse connector
Signed-off-by: Sergey Kiselev <skiselev@gmail.com>
Parts:
- removed R10, R2, R9: 10k, My_Components:Res_Axial_L6.3mm_D2.5mm_P10.16mm_Horizontal
- added C13: 47pF, My_Components:Cap_Cer_508, F.Cu at (175.3, 24.4)
- added C16: 47pF, My_Components:Cap_Cer_508, F.Cu at (175.3, 27.0)
- added JP11: IRQ12: ISA/Mouse, My_Components:Conn_Pin_Header_3x1_2.54mm, F.Cu at (130.8, 128.6)
- added L3: Ferrite, My_Components:L_Ferrite_1016, F.Cu at (188.0, 27.0)
- added L4: Ferrite, My_Components:L_Ferrite_1016, F.Cu at (188.0, 23.5)
- added RP8: 10k, My_Components:Conn_SIL5, F.Cu at (180.3, 21.9)
- J1: value KEYBOARD -> PS/2 Dual Port; footprint My_Components:Conn_DIN_5pin -> My_Components:Conn_Mini_DIN_6pin
- L1, L2: footprint My_Components:Res_1016 -> My_Components:L_Ferrite_1016
- R8: value 470 -> 10k; footprint My_Components:Res_Axial_L6.3mm_D2.5mm_P10.16mm_Horizontal -> My_Components:Res_762
- moved C47 43.4 mm to (182.9, 35.6), turned to -90 degrees
- moved C19 43.2 mm to (167.6, 27.0), turned to 0 degrees
- moved R8 21.7 mm to (166.7, 21.9), turned to 0 degrees
- moved C1 19.5 mm to (190.5, 47.3)
- moved C11 18.2 mm to (167.6, 24.4), turned to 0 degrees
- moved U2 14.5 mm to (158.8, 40.6)
- moved L1 12.2 mm to (188.0, 20.0), turned to 0 degrees
- moved L2 8.52 mm to (188.0, 16.5), turned to 0 degrees
- moved C15 6.10 mm to (175.3, 19.4), turned to 180 degrees
- moved C12 4.41 mm to (175.3, 21.9), turned to 180 degrees
- moved JP2 2.54 mm to (183.5, 49.5)
Connections:
- net Net-(C12-Pad1) renamed /Memory, BIOS, Keyboard, RTC/KBCI
- net Net-(U1-Pad37) renamed /Memory, BIOS, Keyboard, RTC/KBCO
- net Net-(U1-Pad38) renamed /Memory, BIOS, Keyboard, RTC/KBDO
- C15 pad 1: Net-(C15-Pad1) -> /Memory, BIOS, Keyboard, RTC/KBDI
- J1 pad 1: Net-(J1-Pad1) -> /Memory, BIOS, Keyboard, RTC/KB_DATA
- J1 pad 2: Net-(J1-Pad2) -> /Memory, BIOS, Keyboard, RTC/MS_DATA
- J1 pad 3: unconnected-(J1-Pad3) -> GND
- J1 pad 4: GND -> VCC
- J1 pad 5: VCC -> /Memory, BIOS, Keyboard, RTC/KB_CLOCK
- L1 pad 2: Net-(J1-Pad1) -> /Memory, BIOS, Keyboard, RTC/KB_CLOCK
- L2 pad 1: Net-(C15-Pad1) -> /Memory, BIOS, Keyboard, RTC/KBDI
- L2 pad 2: Net-(J1-Pad2) -> /Memory, BIOS, Keyboard, RTC/KB_DATA
- R8 pad 1: VCC -> Net-(U1-Pad2)
- R8 pad 2: Net-(R8-Pad2) -> GND
- U1 pad 2: KBC_CLK -> Net-(U1-Pad2)
- U1 pad 23: unconnected-(U1-Pad23) -> /Memory, BIOS, Keyboard, RTC/MSD0
- U1 pad 24: unconnected-(U1-Pad24) -> /Memory, BIOS, Keyboard, RTC/MSC0
- U1 pad 27: unconnected-(U1-Pad27) -> /Memory, BIOS, Keyboard, RTC/KBDI
- U1 pad 28: unconnected-(U1-Pad28) -> /Memory, BIOS, Keyboard, RTC/MSDI
- U1 pad 3: Net-(R8-Pad2) -> KBC_CLK
- U1 pad 36: unconnected-(U1-Pad36) -> KBC_IRQ12
- U1 pad 39: Net-(C15-Pad1) -> /Memory, BIOS, Keyboard, RTC/MSCI
- U2 pad 10: Net-(R2-Pad2) -> /Memory, BIOS, Keyboard, RTC/KBDI
- U2 pad 12: Net-(C15-Pad1) -> /Memory, BIOS, Keyboard, RTC/MSCI
- U2 pad 13: Net-(R2-Pad2) -> /Memory, BIOS, Keyboard, RTC/MSC0
- U2 pad 3: KBC_CLK -> /Memory, BIOS, Keyboard, RTC/MSD0
- U2 pad 4: Net-(R8-Pad2) -> /Memory, BIOS, Keyboard, RTC/MSDI
- U9 pad 200: IRQ12 -> IRQ12_JP
Routing:
- net KBC_IRQ12: track 0.00 -> 144.6 mm, vias 0 -> 2
- net /Memory, BIOS, Keyboard, RTC/KBDI: track 0.00 -> 80.7 mm, vias 0 -> 1
- net /Memory, BIOS, Keyboard, RTC/MSDI: track 0.00 -> 75.6 mm, vias 0 -> 1
- net /Memory, BIOS, Keyboard, RTC/MSD0: track 0.00 -> 65.4 mm, vias 0 -> 1
- net /Memory, BIOS, Keyboard, RTC/MSC0: track 0.00 -> 55.8 mm, vias 0 -> 1
- net /Memory, BIOS, Keyboard, RTC/MSCI: track 0.00 -> 33.7 mm
- net Net-(C15-Pad1): track 31.8 -> 0.00 mm
- net Net-(R2-Pad2): track 29.1 -> 0.00 mm
- net Net-(J1-Pad2): track 28.7 -> 0.00 mm
- net Net-(J1-Pad1): track 26.8 -> 0.00 mm
- net /Memory, BIOS, Keyboard, RTC/KBCI: track 28.1 -> 53.6 mm, vias 0 -> 1
- net /Memory, BIOS, Keyboard, RTC/KBCO: track 13.0 -> 37.3 mm, vias 0 -> 1
- net IRQ12: track 139.6 -> 120.7 mm, vias 1 -> 0
- net RESET: track 202.2 -> 183.6 mm
- net /Memory, BIOS, Keyboard, RTC/MS_CLOCK: track 0.00 -> 18.5 mm
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Other:
- board text added: "386SX Motherboard Based on SARC RC2016 Chipset Version 1.3 - Copyright (C) 2024 Sergey Kiselev https://github.com/skiselev/mb386sx-rc2016 Based on the M396F motherboard replica by Marco Both: https://github.com/Marco-Both/M396F-Replika"
- board text removed: "386SX Motherboard Based on SARC RC2016 Chipset Version 1.2 - Copyright (C) 2024 Sergey Kiselev https://github.com/skiselev/mb386sx-rc2016 Based on the M396F motherboard replica by Marco Both: https://github.com/Marco-Both/M396F-Replika"
