File: KiCad/bios_kbc_rtc.kicad_sch (KiCad schematic)
At the start: 44 parts, among them J1 PS/2 Dual Port, U1 8242KBD, U10 BANK0, U11 BANK0, U12 BANK1, U13 BANK1, U2 74HC05, U3 SST39SF010A, U4 DS12885, Y2 32768Hz

Commit message: Version 1.9: Add pin headers for the CPU
Other:
- company: (none) -> Copyright (C) 2024-2026 Sergey Kiselev
- title: (none) -> 386SX Motherboard Based on SARC RC2016 Chipset
Changed lines of the file:
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@@
 (kicad_sch (version 20211123) (generator eeschema)
   (paper "A3")
+  (title_block
+    (title "386SX Motherboard Based on SARC RC2016 Chipset")
+    (date "2026-01-09")
+    (rev "1.9")
+    (company "Copyright (C) 2024-2026 Sergey Kiselev")
+    (comment 1 "https://github.com/Marco-Both/M396F-Replika")
+    (comment 2 "Based on the M396F motherboard replica by Marco Both:")
+    (comment 3 "https://github.com/skiselev/mb386sx-rc2016")
+  )
   (junction (at 327.66 106.68) (diameter 0) (color 0 0 0 0)
   )
@@
   (symbol (lib_id "power:GND") (at 73.66 241.3 0) (unit 1)
     (in_bom yes) (on_board yes)
-    (property "Reference" "#PWR?" (id 0) (at 73.66 247.65 0)
+    (property "Reference" "#PWR0141" (id 0) (at 73.66 247.65 0)
       (effects (font (size 1.27 1.27)) hide)
     )

Commit message: Version 2.1: Reorder component references; Update silkscreen; Add signal names on the back silkscreen
Parts:
- renumbered C11 to C3, C66 to C4, C12 to C5, C15 to C6, C13 to C7, C16 to C8, U13 to J10, J1 to J11, U10 to J7, U11 to J8, U12 to J9, R38 to R1, R43 to R10, R44 to R11, R45 to R12, R18 to R16, R50 to R18, R51 to R19, R39 to R2, R52 to R20, R53 to R21, R40 to R3, R8 to R37, R41 to R4, R46 to R5, R47 to R6, R48 to R7, R49 to R8, R42 to R9, RP8 to RN5, U1 to U5, U3 to U6, U2 to U7
