File: KiCad/bios_kbc_rtc.kicad_sch (KiCad schematic)
At the start: 44 parts, among them J1 BANK0, J11 PS/2 Dual Port, J2 BANK0, J3 BANK1, J4 BANK1, U4 DS12885, U5 8242KBD, U6 SST39SF010A, U7 74HC05, Y2 32768Hz

Commit message: Add a polyfuse for the PS/2 port
Parts:
- removed C4: 47pF, My_Components:Cap_Cer_508, symbol Device:C
- added F1: 1.1A, My_Components:Cap_Cer_508, symbol Device:Polyfuse_Small
- renumbered C5 to C4, C6 to C5, C7 to C6, C8 to C7
Connections:
- net VCC: now also F1.2; no longer J11.4
- net ~{MCAS0} renamed ~{CAS0}
- net ~{MCAS1} renamed ~{CAS1}
- net ~{MCAS2} renamed ~{CAS2}
- net ~{MCAS3} renamed ~{CAS3}
- net ~{MRAS01} renamed ~{RAS01}
- net ~{MRAS23} renamed ~{RAS23}
- new net: F1.1, J11.4
Changed lines of the file:
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@@
   (title_block
     (title "386SX Motherboard Based on SARC RC2016 Chipset")
-    (date "2026-02-17")
+    (date "2026-02-18")
     (rev "2.2")
     (company "Copyright (C) 2024-2026 Sergey Kiselev")
@@
   (junction (at 304.8 81.28) (diameter 0) (color 0 0 0 0)
   )
-  (junction (at 213.36 101.6) (diameter 0) (color 0 0 0 0)
-  )
   (junction (at 304.8 68.58) (diameter 0) (color 0 0 0 0)
   )
@@
     (stroke (width 0) (type default) (color 0 0 0 0))
   )
+  (wire (pts (xy 396.24 49.53) (xy 396.24 54.61))
+    (stroke (width 0) (type default) (color 0 0 0 0))
+  )
   (wire (pts (xy 30.48 200.66) (xy 40.64 200.66))
     (stroke (width 0) (type default) (color 0 0 0 0))
@@
     (stroke (width 0) (type default) (color 0 0 0 0))
   )
-  (wire (pts (xy 213.36 101.6) (xy 218.44 101.6))
-    (stroke (width 0) (type default) (color 0 0 0 0))
-  )
   (wire (pts (xy 304.8 58.42) (xy 304.8 68.58))
     (stroke (width 0) (type default) (color 0 0 0 0))
@@
     (stroke (width 0) (type default) (color 0 0 0 0))
   )
-  (wire (pts (xy 208.28 101.6) (xy 213.36 101.6))
+  (wire (pts (xy 208.28 101.6) (xy 218.44 101.6))
     (stroke (width 0) (type default) (color 0 0 0 0))
   )
@@
     (stroke (width 0) (type default) (color 0 0 0 0))
   )
-  (wire (pts (xy 213.36 101.6) (xy 213.36 104.14))
-    (stroke (width 0) (type default) (color 0 0 0 0))
-  )
   (wire (pts (xy 170.18 246.38) (xy 157.48 246.38))
     (stroke (width 0) (type default) (color 0 0 0 0))
@@
     (stroke (width 0) (type default) (color 0 0 0 0))
   )
-  (wire (pts (xy 213.36 114.3) (xy 213.36 111.76))
-    (stroke (width 0) (type default) (color 0 0 0 0))
-  )
   (wire (pts (xy 40.64 104.14) (xy 38.1 104.14))
     (stroke (width 0) (type default) (color 0 0 0 0))
@@
     (stroke (width 0) (type default) (color 0 0 0 0))
   )
-  (wire (pts (xy 396.24 63.5) (xy 396.24 96.52))
+  (wire (pts (xy 396.24 59.69) (xy 396.24 96.52))
     (stroke (width 0) (type default) (color 0 0 0 0))
   )
@@
     )
   )
-  (global_label "~{MRAS23}" (shape input) (at 266.7 254 180) (fields_autoplaced)
+  (global_label "~{RAS23}" (shape input) (at 266.7 254 180) (fields_autoplaced)
     (effects (font (size 1.27 1.27)) (justify right))
-    (property "Intersheet References" "${INTERSHEET_REFS}" (id 0) (at 256.8483 253.9206 0)
+    (property "Intersheet References" "${INTERSHEET_REFS}" (id 0) (at 258.2998 253.9206 0)
       (effects (font (size 1.27 1.27)) (justify right) hide)
     )
@@
     )
   )
-  (global_label "~{MCAS2}" (shape input) (at 226.06 261.62 180) (fields_autoplaced)
+  (global_label "~{CAS2}" (shape input) (at 226.06 261.62 180) (fields_autoplaced)
     (effects (font (size 1.27 1.27)) (justify right))
-    (property "Intersheet References" "${INTERSHEET_REFS}" (id 0) (at 217.4179 261.5406 0)
+    (property "Intersheet References" "${INTERSHEET_REFS}" (id 0) (at 218.8693 261.5406 0)
       (effects (font (size 1.27 1.27)) (justify right) hide)
     )
@@
     )
   )
-  (global_label "~{MRAS01}" (shape input) (at 266.7 246.38 180) (fields_autoplaced)
+  (global_label "~{RAS01}" (shape input) (at 266.7 246.38 180) (fields_autoplaced)
     (effects (font (size 1.27 1.27)) (justify right))
-    (property "Intersheet References" "${INTERSHEET_REFS}" (id 0) (at 256.8483 246.3006 0)
+    (property "Intersheet References" "${INTERSHEET_REFS}" (id 0) (at 258.2998 246.3006 0)
       (effects (font (size 1.27 1.27)) (justify right) hide)
     )
@@
     )
   )
-  (global_label "~{MCAS0}" (shape input) (at 226.06 246.38 180) (fields_autoplaced)
+  (global_label "~{CAS0}" (shape input) (at 226.06 246.38 180) (fields_autoplaced)
     (effects (font (size 1.27 1.27)) (justify right))
-    (property "Intersheet References" "${INTERSHEET_REFS}" (id 0) (at 217.4179 246.3006 0)
+    (property "Intersheet References" "${INTERSHEET_REFS}" (id 0) (at 218.8693 246.3006 0)
       (effects (font (size 1.27 1.27)) (justify right) hide)
     )
@@
     )
   )
-  (global_label "~{MCAS3}" (shape input) (at 226.06 269.24 180) (fields_autoplaced)
+  (global_label "~{CAS3}" (shape input) (at 226.06 269.24 180) (fields_autoplaced)
     (effects (font (size 1.27 1.27)) (justify right))
-    (property "Intersheet References" "${INTERSHEET_REFS}" (id 0) (at 217.4179 269.1606 0)
+    (property "Intersheet References" "${INTERSHEET_REFS}" (id 0) (at 218.8693 269.1606 0)
       (effects (font (size 1.27 1.27)) (justify right) hide)
     )
@@
     )
   )
-  (global_label "~{MCAS1}" (shape input) (at 226.06 254 180) (fields_autoplaced)
+  (global_label "~{CAS1}" (shape input) (at 226.06 254 180) (fields_autoplaced)
     (effects (font (size 1.27 1.27)) (justify right))
-    (property "Intersheet References" "${INTERSHEET_REFS}" (id 0) (at 217.4179 253.9206 0)
+    (property "Intersheet References" "${INTERSHEET_REFS}" (id 0) (at 218.8693 253.9206 0)
       (effects (font (size 1.27 1.27)) (justify right) hide)
     )
@@
     (pin "1")
   )
-  (symbol (lib_id "power:VCC") (at 396.24 63.5 0) (unit 1)
+  (symbol (lib_id "power:VCC") (at 396.24 49.53 0) (unit 1)
     (in_bom yes) (on_board yes)
-    (property "Reference" "#PWR0195" (id 0) (at 396.24 67.31 0)
+    (property "Reference" "#PWR0195" (id 0) (at 396.24 53.34 0)
       (effects (font (size 1.27 1.27)) hide)
     )
-    (property "Value" "VCC" (id 1) (at 396.24 59.69 0))
-    (property "Footprint" "" (id 2) (at 396.24 63.5 0)
+    (property "Value" "VCC" (id 1) (at 396.24 45.72 0))
+    (property "Footprint" "" (id 2) (at 396.24 49.53 0)
       (effects (font (size 1.27 1.27)) hide)
     )
-    (property "Datasheet" "" (id 3) (at 396.24 63.5 0)
+    (property "Datasheet" "" (id 3) (at 396.24 49.53 0)
       (effects (font (size 1.27 1.27)) hide)
     )
@@
   (symbol (lib_id "Device:C") (at 337.82 113.03 0) (unit 1)
     (in_bom yes) (on_board yes)
-    (property "Reference" "C7" (id 0) (at 340.36 111.76 0)
+    (property "Reference" "C6" (id 0) (at 340.36 111.76 0)
       (effects (font (size 1.27 1.27)) (justify left))
     )
@@
     (pin "9")
   )
-  (symbol (lib_id "Device:C") (at 213.36 107.95 0) (unit 1)
-    (in_bom yes) (on_board yes) (fields_autoplaced)
-    (property "Reference" "C4" (id 0) (at 217.17 106.6799 0)
-      (effects (font (size 1.27 1.27)) (justify left))
-    )
-    (property "Value" "47pF" (id 1) (at 217.17 109.2199 0)
-      (effects (font (size 1.27 1.27)) (justify left))
-    )
-    (property "Footprint" "My_Components:Cap_Cer_508" (id 2) (at 214.3252 111.76 0)
-      (effects (font (size 1.27 1.27)) hide)
-    )
-    (property "Datasheet" "~" (id 3) (at 213.36 107.95 0)
-      (effects (font (size 1.27 1.27)) hide)
-    )
-    (pin "1")
-    (pin "2")
-  )
   (symbol (lib_id "Device:L_Ferrite") (at 354.33 93.98 90) (unit 1)
     (in_bom yes) (on_board yes)
@@
     (pin "1")
   )
-  (symbol (lib_id "power:GND") (at 213.36 114.3 0) (unit 1)
-    (in_bom yes) (on_board yes)
-    (property "Reference" "#PWR0218" (id 0) (at 213.36 120.65 0)
-      (effects (font (size 1.27 1.27)) hide)
-    )
-    (property "Value" "GND" (id 1) (at 213.36 118.11 0))
-    (property "Footprint" "" (id 2) (at 213.36 114.3 0)
-      (effects (font (size 1.27 1.27)) hide)
-    )
-    (property "Datasheet" "" (id 3) (at 213.36 114.3 0)
-      (effects (font (size 1.27 1.27)) hide)
-    )
-    (pin "1")
-  )
   (symbol (lib_id "Device:C") (at 347.98 113.03 0) (unit 1)
     (in_bom yes) (on_board yes)
-    (property "Reference" "C8" (id 0) (at 350.52 111.76 0)
+    (property "Reference" "C7" (id 0) (at 350.52 111.76 0)
       (effects (font (size 1.27 1.27)) (justify left))
     )
@@
   (symbol (lib_id "Device:C") (at 327.66 113.03 0) (unit 1)
     (in_bom yes) (on_board yes)
-    (property "Reference" "C6" (id 0) (at 330.2 111.76 0)
+    (property "Reference" "C5" (id 0) (at 330.2 111.76 0)
       (effects (font (size 1.27 1.27)) (justify left))
     )
@@
   (symbol (lib_id "Device:C") (at 317.5 113.03 0) (unit 1)
     (in_bom yes) (on_board yes)
-    (property "Reference" "C5" (id 0) (at 320.04 111.76 0)
+    (property "Reference" "C4" (id 0) (at 320.04 111.76 0)
       (effects (font (size 1.27 1.27)) (justify left))
     )
@@
       (effects (font (size 1.27 1.27)) hide)
     )
+    (pin "1")
+    (pin "2")
+  )
+  (symbol (lib_id "Device:Polyfuse_Small") (at 396.24 57.15 180) (unit 1)
+    (in_bom yes) (on_board yes) (fields_autoplaced)
+    (property "Reference" "F1" (id 0) (at 398.78 55.8799 0)
+      (effects (font (size 1.27 1.27)) (justify right))
+    )
+    (property "Value" "1.1A" (id 1) (at 398.78 58.4199 0)
+      (effects (font (size 1.27 1.27)) (justify right))
+    )
+    (property "Footprint" "My_Components:Cap_Cer_508" (id 2) (at 394.97 52.07 0)
+      (effects (font (size 1.27 1.27)) (justify left) hide)
+    )
+    (property "Datasheet" "~" (id 3) (at 396.24 57.15 0)
+      (effects (font (size 1.27 1.27)) hide)
+    )

Commit message: Add version 2.3 files
Parts:
- J11: symbol Connector:Mini-DIN-6 -> my_components:Conn_Mini-DIN-6_Shielded
Connections:
- net GND: now also J11.SH
Changed lines of the file:
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@@
   (title_block
     (title "386SX Motherboard Based on SARC RC2016 Chipset")
-    (date "2026-02-18")
-    (rev "2.2")
+    (date "2026-02-26")
+    (rev "2.3")
     (company "Copyright (C) 2024-2026 Sergey Kiselev")
     (comment 1 "https://github.com/Marco-Both/M396F-Replika")
@@
     (stroke (width 0) (type default) (color 0 0 0 0))
   )
-  (wire (pts (xy 373.38 96.52) (xy 373.38 106.68))
+  (wire (pts (xy 373.38 96.52) (xy 373.38 119.38))
     (stroke (width 0) (type default) (color 0 0 0 0))
   )
@@
   )
   (wire (pts (xy 198.12 213.36) (xy 198.12 215.9))
+    (stroke (width 0) (type default) (color 0 0 0 0))
+  )
+  (wire (pts (xy 383.54 119.38) (xy 383.54 106.68))
     (stroke (width 0) (type default) (color 0 0 0 0))
   )
@@
     (pin "2")
   )
-  (symbol (lib_id "power:GND") (at 373.38 106.68 0) (unit 1)
-    (in_bom yes) (on_board yes)
-    (property "Reference" "#PWR0188" (id 0) (at 373.38 113.03 0)
-      (effects (font (size 1.27 1.27)) hide)
-    )
-    (property "Value" "GND" (id 1) (at 373.38 110.49 0))
-    (property "Footprint" "" (id 2) (at 373.38 106.68 0)
-      (effects (font (size 1.27 1.27)) hide)
-    )
-    (property "Datasheet" "" (id 3) (at 373.38 106.68 0)
+  (symbol (lib_id "power:GND") (at 373.38 119.38 0) (unit 1)
+    (in_bom yes) (on_board yes)
+    (property "Reference" "#PWR0188" (id 0) (at 373.38 125.73 0)
+      (effects (font (size 1.27 1.27)) hide)
+    )
+    (property "Value" "GND" (id 1) (at 373.38 123.19 0))
+    (property "Footprint" "" (id 2) (at 373.38 119.38 0)
+      (effects (font (size 1.27 1.27)) hide)
+    )
+    (property "Datasheet" "" (id 3) (at 373.38 119.38 0)
       (effects (font (size 1.27 1.27)) hide)
     )
@@
     (pin "1")
     (pin "2")
+  )
+  (symbol (lib_id "power:GND") (at 383.54 119.38 0) (unit 1)
+    (in_bom yes) (on_board yes)
+    (property "Reference" "#PWR0157" (id 0) (at 383.54 125.73 0)
+      (effects (font (size 1.27 1.27)) hide)
+    )
+    (property "Value" "GND" (id 1) (at 383.54 123.19 0))
+    (property "Footprint" "" (id 2) (at 383.54 119.38 0)
+      (effects (font (size 1.27 1.27)) hide)
+    )
+    (property "Datasheet" "" (id 3) (at 383.54 119.38 0)
+      (effects (font (size 1.27 1.27)) hide)
+    )
+    (pin "1")
   )
   (symbol (lib_id "power:GND") (at 55.88 241.3 0) (unit 1)
@@
     (pin "2")
   )
-  (symbol (lib_id "Connector:Mini-DIN-6") (at 383.54 96.52 0) (mirror y) (unit 1)
+  (symbol (lib_id "my_components:Conn_Mini-DIN-6_Shielded") (at 383.54 96.52 0) (mirror y) (unit 1)
     (in_bom yes) (on_board yes) (fields_autoplaced)
     (property "Reference" "J11" (id 0) (at 383.5223 86.36 0))
@@
     (pin "5")
     (pin "6")
+    (pin "SH")
   )
   (symbol (lib_id "power:GND") (at 101.6 67.31 0) (unit 1)
