File: KiCad/isa_slots_power.kicad_sch (KiCad schematic)
At the start: 82 parts, among them J10 BUSAT_HOST, J12 Power, J5 BUSAT_HOST, J6 BUSAT_HOST, J7 BUSAT_HOST, J8 BUSAT_HOST, J9 BUSAT_HOST, U10 LM7905, U8 74HCT14, U9 74HCT74

Commit message: Add a polyfuse for the PS/2 port
Parts:
- removed C50, C51, C52, C53, C54, C55, C56, C57, C58, C59, C60, C61: DNP, My_Components:Cap_Cer_508, symbol Device:C
- renumbered C11 to C10, C12 to C11, C13 to C12, C14 to C13, C15 to C14, C16 to C15, C17 to C16, C18 to C17, C19 to C18, C20 to C19, C21 to C20, C23 to C22, C24 to C23, C25 to C24, C26 to C25, C27 to C26, C28 to C27, C29 to C28, C30 to C29, C31 to C30, C32 to C31, C33 to C32, C34 to C33, C35 to C34, C36 to C35, C37 to C36, C38 to C37, C39 to C38, C40 to C39, C41 to C40, C42 to C41, C43 to C42, C44 to C43, C45 to C44, C46 to C45, C47 to C46, C48 to C47, C49 to C48
Other:
- moved on the sheet: D1, H1, H2, H3, H4, H5, H6, H7, R27, R30, R35, R36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
